File: Macroboard.sch (KiCad schematic (older format))
At the start: 34 parts, among them SW1 SW_Push, U1 ATmega32U4-AU, Y1 16MHz

Commit message: pcb base
Parts:
- MX1, MX2, MX3, MX4, MX5, MX6, MX7, MX8, MX9: footprint MX_Only:MXOnly-1.5U-NoLED -> MX_Only:MXOnly-1U-NoLED
Changed lines of the file:
@@
 F 0 "MX1" H 8133 1323 60  0000 C CNN
 F 1 "MX-NoLED" H 8133 1249 20  0000 C CNN
-F 2 "MX_Only:MXOnly-1.5U-NoLED" H 7475 1075 60  0001 C CNN
+F 2 "MX_Only:MXOnly-1U-NoLED" H 7475 1075 60  0001 C CNN
 F 3 "" H 7475 1075 60  0001 C CNN
 	1    8100 1100
@@
 F 0 "MX2" H 8633 1323 60  0000 C CNN
 F 1 "MX-NoLED" H 8633 1249 20  0000 C CNN
-F 2 "MX_Only:MXOnly-1.5U-NoLED" H 7975 1075 60  0001 C CNN
+F 2 "MX_Only:MXOnly-1U-NoLED" H 7975 1075 60  0001 C CNN
 F 3 "" H 7975 1075 60  0001 C CNN
 	1    8600 1100
@@
 F 0 "MX3" H 9133 1323 60  0000 C CNN
 F 1 "MX-NoLED" H 9133 1249 20  0000 C CNN
-F 2 "MX_Only:MXOnly-1.5U-NoLED" H 8475 1075 60  0001 C CNN
+F 2 "MX_Only:MXOnly-1U-NoLED" H 8475 1075 60  0001 C CNN
 F 3 "" H 8475 1075 60  0001 C CNN
 	1    9100 1100
@@
 F 0 "MX4" H 8133 2323 60  0000 C CNN
 F 1 "MX-NoLED" H 8133 2249 20  0000 C CNN
-F 2 "MX_Only:MXOnly-1.5U-NoLED" H 7475 2075 60  0001 C CNN
+F 2 "MX_Only:MXOnly-1U-NoLED" H 7475 2075 60  0001 C CNN
 F 3 "" H 7475 2075 60  0001 C CNN
 	1    8100 2100
@@
 F 0 "MX5" H 8633 2323 60  0000 C CNN
 F 1 "MX-NoLED" H 8633 2249 20  0000 C CNN
-F 2 "MX_Only:MXOnly-1.5U-NoLED" H 7975 2075 60  0001 C CNN
+F 2 "MX_Only:MXOnly-1U-NoLED" H 7975 2075 60  0001 C CNN
 F 3 "" H 7975 2075 60  0001 C CNN
 	1    8600 2100
@@
 F 0 "MX6" H 9133 2323 60  0000 C CNN
 F 1 "MX-NoLED" H 9133 2249 20  0000 C CNN
-F 2 "MX_Only:MXOnly-1.5U-NoLED" H 8475 2075 60  0001 C CNN
+F 2 "MX_Only:MXOnly-1U-NoLED" H 8475 2075 60  0001 C CNN
 F 3 "" H 8475 2075 60  0001 C CNN
 	1    9100 2100
@@
 F 0 "MX7" H 8133 3323 60  0000 C CNN
 F 1 "MX-NoLED" H 8133 3249 20  0000 C CNN
-F 2 "MX_Only:MXOnly-1.5U-NoLED" H 7475 3075 60  0001 C CNN
+F 2 "MX_Only:MXOnly-1U-NoLED" H 7475 3075 60  0001 C CNN
 F 3 "" H 7475 3075 60  0001 C CNN
 	1    8100 3100
@@
 F 0 "MX8" H 8633 3323 60  0000 C CNN
 F 1 "MX-NoLED" H 8633 3249 20  0000 C CNN
-F 2 "MX_Only:MXOnly-1.5U-NoLED" H 7975 3075 60  0001 C CNN
+F 2 "MX_Only:MXOnly-1U-NoLED" H 7975 3075 60  0001 C CNN
 F 3 "" H 7975 3075 60  0001 C CNN
 	1    8600 3100
@@
 F 0 "MX9" H 9133 3323 60  0000 C CNN
 F 1 "MX-NoLED" H 9133 3249 20  0000 C CNN
-F 2 "MX_Only:MXOnly-1.5U-NoLED" H 8475 3075 60  0001 C CNN
+F 2 "MX_Only:MXOnly-1U-NoLED" H 8475 3075 60  0001 C CNN
 F 3 "" H 8475 3075 60  0001 C CNN
 	1    9100 3100
