File: Macroboard.kicad_pcb (KiCad board)
At the start: 2 copper layers, 76.2 x 84.9 mm, 49 parts, among them Q1 2N7002, SW1 SW_Push, U1 ATmega32U4-AU, Y1 16MHz

Commit message: small fixes
Routing:
- net VCC: track 14.4 -> 6.78 mm
Changed lines of the file:
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@@
     (thickness 1.6)
     (drawings 15)
-    (tracks 421)
+    (tracks 419)
     (zones 0)
     (modules 49)
@@
   )
   (setup
-    (last_trace_width 0.254)
+    (last_trace_width 0.381)
+    (user_trace_width 0.381)
     (trace_clearance 0.2)
     (zone_clearance 0.508)
@@
     (visible_elements 7FFFFFFF)
     (pcbplotparams
-      (layerselection 0x010fc_ffffffff)
-      (usegerberextensions false)
+      (layerselection 0x010f0_ffffffff)
+      (usegerberextensions true)
       (usegerberattributes false)
       (usegerberadvancedattributes false)
@@
       (plotinvisibletext false)
       (padsonsilk false)
-      (subtractmaskfromsilk false)
+      (subtractmaskfromsilk true)
       (outputformat 1)
       (mirror false)
-      (drillshape 1)
+      (drillshape 0)
       (scaleselection 1)
-      (outputdirectory ""))
+      (outputdirectory "Gerbers"))
   )
   (net 0 "")
@@
   (gr_arc (start 274.6375 65.0875) (end 276.225 65.0875) (angle -90) (layer Edge.Cuts) (width 0.05))
   (gr_arc (start 202.40625 65.0875) (end 202.40625 63.5) (angle -90) (layer Edge.Cuts) (width 0.05))
-  (segment (start 253.492 113.31226) (end 253.492 95.85325) (width 0.254) (layer F.Cu) (net 12))
-  (segment (start 253.492 132.48926) (end 253.492 115.03025) (width 0.254) (layer F.Cu) (net 12))
-  (segment (start 234.442 132.48926) (end 234.442 115.03025) (width 0.254) (layer F.Cu) (net 11))
-  (segment (start 234.315 113.31226) (end 234.315 95.85325) (width 0.254) (layer F.Cu) (net 11))
   (segment (start 245.796 70.021) (end 245.131 69.356) (width 0.381) (layer B.Cu) (net 1))
   (segment (start 245.796 73.929) (end 245.796 70.021) (width 0.381) (layer B.Cu) (net 1))
@@
   (via (at 268.2875 107.95) (size 0.8) (drill 0.4) (layers F.Cu B.Cu) (net 5))
   (segment (start 265.1125 107.95) (end 268.2875 107.95) (width 0.381) (layer F.Cu) (net 5))
-  (segment (start 268.2875 141.2875) (end 268.2875 127) (width 0.381) (layer B.Cu) (net 5))
-  (segment (start 263.525 146.05) (end 268.2875 141.2875) (width 0.381) (layer B.Cu) (net 5))
   (segment (start 219.86875 144.4625) (end 219.86875 145.25625) (width 0.381) (layer B.Cu) (net 5))
   (segment (start 219.86875 145.25625) (end 220.6625 146.05) (width 0.381) (layer B.Cu) (net 5))
@@
   (segment (start 258.05 145.3375) (end 258.7625 146.05) (width 0.381) (layer B.Cu) (net 5))
   (segment (start 239.7125 146.05) (end 258.7625 146.05) (width 0.381) (layer B.Cu) (net 5))
-  (segment (start 258.7625 146.05) (end 263.525 146.05) (width 0.381) (layer B.Cu) (net 5))
   (segment (start 268.2875 107.95) (end 268.2875 82.55) (width 0.381) (layer B.Cu) (net 5))
   (segment (start 262.1915 76.454) (end 254.889 76.454) (width 0.381) (layer B.Cu) (net 5))
@@
   (segment (start 238.76 70.993) (end 238.633 70.866) (width 0.381) (layer B.Cu) (net 5))
   (segment (start 238.76 71.501) (end 238.76 70.993) (width 0.381) (layer B.Cu) (net 5))
+  (segment (start 268.2875 139.1285) (end 268.2875 138.3665) (width 0.254) (layer B.Cu) (net 5))
+  (segment (start 268.2875 139.1285) (end 268.2875 127) (width 0.381) (layer B.Cu) (net 5))
+  (segment (start 263.525 143.8275) (end 268.2875 139.065) (width 0.381) (layer B.Cu) (net 5))
+  (segment (start 258.7625 146.05) (end 261.3025 146.05) (width 0.381) (layer B.Cu) (net 5))
+  (segment (start 261.3025 146.05) (end 263.525 143.8275) (width 0.381) (layer B.Cu) (net 5))
   (segment (start 245.71775 100.457) (end 227.35725 100.457) (width 0.254) (layer B.Cu) (net 6))
   (segment (start 246.0625 99.40825) (end 246.0625 100.11225) (width 0.254) (layer B.Cu) (net 6))
@@
   (segment (start 223.04375 138.90625) (end 225.425 138.90625) (width 0.254) (layer B.Cu) (net 8))
   (segment (start 225.425 138.90625) (end 245.26875 138.90625) (width 0.254) (layer B.Cu) (net 8))
-  (segment (start 219.761 70.653) (end 217.262 73.152) (width 0.254) (layer B.Cu) (net 9))
-  (segment (start 217.17 73.244) (end 219.761 70.653) (width 0.254) (layer B.Cu) (net 9))
-  (segment (start 217.17 74.549) (end 217.17 73.244) (width 0.254) (layer B.Cu) (net 9))
   (segment (start 219.761 70.653) (end 219.761 69.778) (width 0.254) (layer B.Cu) (net 9))
-  (segment (start 217.179347 73.234653) (end 219.761 70.653) (width 0.254) (layer B.Cu) (net 9))
-  (segment (start 217.179347 73.523653) (end 217.179347 73.234653) (width 0.254) (layer B.Cu) (net 9))
-  (segment (start 216.408 74.295) (end 217.179347 73.523653) (width 0.254) (layer B.Cu) (net 9))
+  (segment (start 219.761 70.942) (end 216.408 74.295) (width 0.381) (layer B.Cu) (net 9))
+  (segment (start 219.761 69.778) (end 219.761 70.942) (width 0.381) (layer B.Cu) (net 9))
   (segment (start 244.49551 90.03349) (end 220.32276 90.03349) (width 0.254) (layer B.Cu) (net 10))
   (segment (start 248.196 86.333) (end 244.49551 90.03349) (width 0.254) (layer B.Cu) (net 10))
@@
   (segment (start 215.265 112.55026) (end 215.265 95.09125) (width 0.254) (layer F.Cu) (net 10))
   (segment (start 215.265 95.09125) (end 220.32276 90.03349) (width 0.254) (layer B.Cu) (net 10))
+  (segment (start 234.442 132.48926) (end 234.442 115.03025) (width 0.254) (layer F.Cu) (net 11))
+  (segment (start 234.315 113.31226) (end 234.315 95.85325) (width 0.254) (layer F.Cu) (net 11))
   (segment (start 248.996 86.333) (end 248.996 85.329) (width 0.254) (layer B.Cu) (net 11))
   (segment (start 244.8415 90.4875) (end 248.996 86.333) (width 0.254) (layer B.Cu) (net 11))
   (segment (start 234.315 95.09125) (end 238.91875 90.4875) (width 0.254) (layer B.Cu) (net 11))
   (segment (start 238.91875 90.4875) (end 244.8415 90.4875) (width 0.254) (layer B.Cu) (net 11))
+  (segment (start 253.492 113.31226) (end 253.492 95.85325) (width 0.254) (layer F.Cu) (net 12))
+  (segment (start 253.492 132.48926) (end 253.492 115.03025) (width 0.254) (layer F.Cu) (net 12))
   (segment (start 249.796 91.52225) (end 249.796 85.329) (width 0.254) (layer B.Cu) (net 12))
   (segment (start 253.365 95.09125) (end 249.796 91.52225) (width 0.254) (layer B.Cu) (net 12))
@@
   (segment (start 260.632 84.681) (end 260.477 84.526) (width 0.254) (layer B.Cu) (net 48))
   (segment (start 261.62 84.681) (end 260.632 84.681) (width 0.254) (layer B.Cu) (net 48))
+  (segment (start 265.607 82.931) (end 265.668 82.87) (width 0.254) (layer B.Cu) (net 49))
+  (segment (start 261.62 82.931) (end 265.607 82.931) (width 0.254) (layer B.Cu) (net 49))
   (segment (start 258.445 142.14475) (end 259.17525 142.875) (width 0.381) (layer B.Cu) (net 50))
   (segment (start 259.17525 142.875) (end 259.55625 142.875) (width 0.381) (layer B.Cu) (net 50))
@@
   (segment (start 262.73125 142.875) (end 263.525 142.875) (width 0.381) (layer B.Cu) (net 50))
   (segment (start 259.55625 142.875) (end 262.73125 142.875) (width 0.381) (layer B.Cu) (net 50))
+  (segment (start 265.938 83.82) (end 266.156602 83.82) (width 0.381) (layer B.Cu) (net 50))
+  (segment (start 263.668 83.82) (end 265.938 83.82) (width 0.381) (layer B.Cu) (net 50))
+  (segment (start 266.954 139.446) (end 266.7 139.7) (width 0.381) (layer B.Cu) (net 50))
+  (segment (start 266.954 84.201) (end 266.954 139.446) (width 0.381) (layer B.Cu) (net 50))
+  (segment (start 265.938 83.82) (end 266.573 83.82) (width 0.381) (layer B.Cu) (net 50))
+  (segment (start 266.573 83.82) (end 266.954 84.201) (width 0.381) (layer B.Cu) (net 50))
   (segment (start 218.2 103.10625) (end 217.805 102.71125) (width 0.254) (layer B.Cu) (net 51))
   (segment (start 218.2 106.3625) (end 218.2 103.10625) (width 0.254) (layer B.Cu) (net 51))
@@
   (via (at 251.61875 144.4625) (size 0.8) (drill 0.4) (layers F.Cu B.Cu) (net 59))
   (via (at 251.61875 141.2875) (size 0.8) (drill 0.4) (layers F.Cu B.Cu) (net 59))
-  (segment (start 265.607 82.931) (end 265.668 82.87) (width 0.254) (layer B.Cu) (net 49))
-  (segment (start 261.62 82.931) (end 265.607 82.931) (width 0.254) (layer B.Cu) (net 49))
-  (segment (start 265.938 83.82) (end 266.156602 83.82) (width 0.381) (layer B.Cu) (net 50))
-  (segment (start 263.668 83.82) (end 265.938 83.82) (width 0.381) (layer B.Cu) (net 50))
-  (segment (start 266.954 139.446) (end 266.7 139.7) (width 0.381) (layer B.Cu) (net 50))
-  (segment (start 266.954 84.201) (end 266.954 139.446) (width 0.381) (layer B.Cu) (net 50))
-  (segment (start 265.938 83.82) (end 266.573 83.82) (width 0.381) (layer B.Cu) (net 50))
-  (segment (start 266.573 83.82) (end 266.954 84.201) (width 0.381) (layer B.Cu) (net 50))
   (zone (net 1) (net_name GND) (layer B.Cu) (hatch edge 0.508)
     (connect_pads (clearance 0.508))
